Commit message: hokuyo LIDAR added

File: src/robot/urdf/robot.xacro (robot description, xacro)
@@ -39,5 +39,5 @@
     <pose>0 0 0 0 0 0</pose>
     <inertial>
-      <mass value="0.35"/>
+      <mass value="5.35"/>
       <origin xyz="0 0 0" rpy="0 0 0"/>
       <inertia
@@ -64,5 +64,5 @@
     <pose>0 0 0 0 0 0</pose>
     <inertial>
-      <mass value="0.35"/>
+      <mass value="5.35"/>
       <origin xyz="0 0 0" rpy="0 0 0"/>
       <inertia
@@ -109,4 +109,29 @@
       </geometry>
       <material name="black"/>
+    </visual>
+  </link>
+<!-- links for sensors -->
+  <link name='hokuyo'>
+    <pose>0 0 0 0 0 0</pose>
+    <inertial>
+      <mass value="1e-5"/>
+      <origin xyz="0 0 0" rpy="0 0 0"/>
+      <inertia
+          ixx="1e-6" ixy="0" ixz="0"
+          iyy="1e-6" iyz="0"
+          izz="1e-6"
+      />
+    </inertial>
+    <collision name='LIDAR_collision'>
+      <origin xyz="0 0 0" rpy="0 0 0"/>
+      <geometry>
+        <mesh filename="package://robot/meshes/hokuyo.dae"/>
+      </geometry>
+    </collision>
+    <visual name='LIDAR_visual'>
+      <origin xyz="0 0 0" rpy="0 0 0"/>
+      <geometry>
+        <mesh filename="package://robot/meshes/hokuyo.dae"/>
+      </geometry>
     </visual>
   </link>
@@ -173,4 +198,9 @@
     <parent link="camera_link"/>
     <child link="camera_link_fake"/>
+  </joint>
+  <joint name="hokuyo_joint" type="fixed">
+    <origin xyz="-0.2 0 0.1" rpy="0 0 0"/>
+    <parent link="robot_body"/>
+    <child link="hokuyo"/>
   </joint>
   <gazebo reference="left_wheel">

Commit message: added LIDAR and extra weight for stability

File: src/robot/urdf/robot.xacro (robot description, xacro)
@@ -200,5 +200,5 @@
   </joint>
   <joint name="hokuyo_joint" type="fixed">
-    <origin xyz="-0.2 0 0.1" rpy="0 0 0"/>
+    <origin xyz="-0.2 0 0.1" rpy="0 0 3.1415"/>
     <parent link="robot_body"/>
     <child link="hokuyo"/>

Commit message: changed URDF to match MediBot Hardware design

File: src/robot/urdf/robot.xacro (robot description, xacro)
@@ -7,5 +7,6 @@
   <link name='robot_footprint'> </link>
   <joint name="robot_footprint_joint" type="fixed">
-    <origin xyz="0 0 0" rpy="0 0 0" />
+    <origin xyz="0 0 0" rpy="1.57 0 3.1415" />
+<!-- x poits towards back of body, y upwards -->
     <parent link="robot_footprint"/>
     <child link="robot_body" />
@@ -15,5 +16,5 @@
     <inertial>
       <mass value="9"/>
-      <origin xyz="0 0 0" rpy=" 1.5707 0 1.5707"/>
+      <origin xyz="0 0 0" rpy=" 0 0 0"/>
       <inertia
           ixx="0.4298" ixy="0" ixz="0"
@@ -23,14 +24,14 @@
     </inertial>
     <collision name='robot_collision'>
-      <origin xyz="0 0 0" rpy=" 1.5707 0 1.5707"/>
+      <origin xyz="0 0 0" rpy=" 0 0 0"/>
       <geometry>
         <!--<box size="1.0 1.0 1.0"/>-->
-        <mesh filename="package://robot/meshes/dingo_for_omni.dae"/>
+        <mesh filename="package://robot/meshes/chassis.dae"/>
       </geometry>
     </collision>
     <visual name='robot_visual'>
-      <origin xyz="0 0 0" rpy=" 1.5707 0 1.5707"/>
-      <geometry>
-        <mesh filename="package://robot/meshes/dingo_for_omni.dae"/>
+      <origin xyz="0 0 0" rpy=" 0 0 0"/>
+      <geometry>
+        <mesh filename="package://robot/meshes/chassis.dae"/>
       </geometry>
     </visual>
@@ -100,5 +101,5 @@
       <origin xyz="0 0 0" rpy="0 0 0"/>
       <geometry>
-        <sphere radius="0.02"/>
+        <sphere radius="0.045"/>
       </geometry>
     </collision>
@@ -106,5 +107,5 @@
       <origin xyz="0 0 0" rpy="0 0 0"/>
       <geometry>
-        <sphere radius="0.02"/>
+        <sphere radius="0.045"/>
       </geometry>
       <material name="black"/>
@@ -136,4 +137,5 @@
     </visual>
   </link>
+  <!--
   <link name='camera_link'>
     <pose>0 0 0 0 0 0</pose>
@@ -160,8 +162,11 @@
     </visual>
   </link>
-  <link name='camera_link_fake'> <!-- To control the face of camera link which will be used as camera, we make an invisible link -->
-  </link>
+-->
+ <!-- To control the face of camera link which will be used as camera, we make an invisible link
+ <link name='camera_link_fake'>
+  </link>
+-->
   <joint type="continuous" name="left_wheel_hinge">
-    <origin xyz="-0.100266 -0.242145 0.03" rpy=" 0 -1.5707 1.5707"/>
+    <origin xyz="0 0 0.27" rpy="0 0 0"/>
     <child link="left_wheel"/>
     <parent link="robot_body"/>
@@ -171,5 +176,5 @@
   </joint>
   <joint type="continuous" name="right_wheel_hinge">
-    <origin xyz="-0.100266 0.242145 0.03" rpy=" 0 -1.5707 1.5707"/>
+    <origin xyz="0 0 -0.27" rpy="0 0 0"/>
     <child link="right_wheel"/>
     <parent link="robot_body"/>
@@ -178,4 +183,5 @@
     <dynamics damping="1.0" friction="1.0"/>
   </joint>
+<!--
   <joint type="fixed" name="camera_link_hinge">
     <origin xyz="-0.285635 0.0 0.05051" rpy="-1.57 0 1.57"/>
@@ -186,6 +192,7 @@
     <dynamics damping="1.0" friction="1.0"/>
   </joint>
+  -->
   <joint type="continuous" name="omni_wheel_hinge">
-    <origin xyz="0.233497 -0.000865 0" rpy="0.000212 -0.118296 -0.001802"/>
+    <origin xyz="0.233497 0 0" rpy="0.000212 -0.118296 -0.001802"/>
     <child link="omni_wheel"/>
     <parent link="robot_body"/>
@@ -194,4 +201,5 @@
     <dynamics damping="1.0" friction="1.0"/>
   </joint>
+  <!--
   <joint name="camera_fake_joint" type="fixed">
     <origin xyz="0 0 0" rpy="-1.57 -1.57 3.14"/>
@@ -199,6 +207,7 @@
     <child link="camera_link_fake"/>
   </joint>
+-->
   <joint name="hokuyo_joint" type="fixed">
-    <origin xyz="-0.2 0 0.1" rpy="0 0 3.1415"/>
+    <origin xyz="-0.409 0.07 0" rpy="-1.57 3.14 0"/>
     <parent link="robot_body"/>
     <child link="hokuyo"/>
